File: LRE_Controller.kicad_sch (KiCad schematic)
At the start: 0 parts

Commit message: Added buck to schematic
Parts:
- added BT1: 5V (Battery_Cell), symbol Device:Battery_Cell
- added C1, C8: 100n, symbol Device:C_Polarized
- added C2, C4: 10u, symbol Device:C_Polarized
- added C3: 22n, symbol Device:C
- added C7: 30p, symbol Device:C_Polarized
- added C9: 215.061, symbol Device:C_Polarized
- added L1: 6.8u, symbol Device:L
- added R1: 52k3, symbol Device:R
- added R2: 100k, symbol Device:R
- added R3: 412k, symbol Device:R
- added R4: 20k, symbol Device:R
- added U1: TPS56A37RPAR, RPA0010A-MFG, symbol Imported_ICs:TPS56A37RPAR
Connections:
- new net: C7.2, R3.2, R4.1, U1.2 (FB)
- new net: C3.2, U1.5 (SS)
- new net: BT1.1 (+), R2.2
- new net: R2.1, U1.4 (PG)
- new net: C8.1, U1.7 (BOOT)
- new net: C8.2, L1.1, U1.6 (SW)
- new net: R1.1, U1.10 (MODE)
- new net +28V: C1.1, C2.1, C4.1, U1.8 (VIN)
- new net GNDA: BT1.2 (-), C1.2, C2.2, C3.1, C4.2, C9.2, R1.2, R4.2, U1.3 (AGND), U1.9 (PGND)
- new net Motor_IN: C7.1, C9.1, L1.2, R3.1
- no-connect marks 0 -> 1
